Commit message: error handler

File: sdv_robot_description/urdf/robot.urdf (robot description, URDF)
Before this commit: robot dasautonomeauto, 4 links, 3 joints
Links:
- link base_link: geometry collision mesh filename=file://$(find sdv_robot_description)/meshes/sdv.stl; visual mesh filename=file://$(find sdv_robot_description)/meshes/sdv.stl

Commit message: lidar uploud

File: sdv_robot_description/urdf/robot.urdf (robot description, URDF)
Before this commit: robot dasautonomeauto, 4 links, 3 joints
Links:
- added link detector_wall
Joints:
- added joint detector_wall_joint: type fixed, parent base_footprint, child detector_wall, origin xyz=0 1.45 1.1 rpy=0 0 0

Commit message: ground plannar added

File: sdv_robot_description/urdf/robot.urdf (robot description, URDF)
Before this commit: robot dasautonomeauto, 5 links, 4 joints
Joints:
- joint velodyne_base_mount_joint: origin xyz=0 0 1.8 rpy=0 0 0 -> xyz=0 0 1.8 rpy=-0.174533 0 0

Commit message: sync lidar imu

File: sdv_robot_description/urdf/robot.urdf (robot description, URDF)
Before this commit: robot dasautonomeauto, 5 links, 4 joints
Links:
- added link vectornav
Joints:
- added joint vectornav_joint: type fixed, parent base_link, child vectornav, origin xyz=0 -0.2 1.8 rpy=0 0 0
