Commit message: zf working

File: sdv_robot_description/urdf/zf_car.urdf (robot description, URDF)
Before this commit: robot dasautonomeauto, 2 links, 1 joints
Links:
- added link base_footprint
Joints:
- added joint base_link_joint: type fixed, parent base_footprint, child chassis_link, origin xyz=0 0 0.5 rpy=0 0 0
